File: CustomKeyboard/CustomKeyboard.kicad_pcb (KiCad board)
At the start: 2 copper layers, 175 parts, among them J1 629105136821, SW1 PEC11H-RotaryEncoderSwitch, U1 ATMEGA32U4-AUR

Commit message: Finished Initial Footprints and started layout
Parts:
- added D47: 1N4148WX-TP, keyboard_fp:SOD323, F.Cu at (87.6, -26.7)
- added D87: 1N4148WX-TP, keyboard_fp:SOD323, F.Cu at (66.2, -23.9)
- added D87: 1N4148WX-TP, keyboard_fp:SOD323, F.Cu at (86.7, -76.4)
- added D88: 1N4148WX-TP, keyboard_fp:SOD323, F.Cu at (86.7, -78.3)
- added KS86: BSP, keyboard_fp:CherryMx, F.Cu at (388.6, -16.5)
- added SW1: PEC11H-RotaryEncoderSwitch, keyboard_fp:PEC11H-RotaryEncoderSwitch, F.Cu at (47.0, 30.5)
- J1: value 629105136821 -> GCT-USB4085; footprint keyboard_fp:629105136821(Wurth USB-BMicro) -> keyboard_fp:USB4085-GF-A
- KS27: renamed from KS26; value SPACE -> SPA
- KS28: renamed from KS27; value INS -> INSERT
- KS5: value LSHIFT -> LSH
- KS6: value LCTRL -> LCTL
- KS65: value UPARR -> UPA
- KS67: value 10 -> 0
- KS72: value LARR -> LAR
- KS74: value 11 -> -
- KS77: value RSHIFT -> RSH
- KS79: value DARR -> DAR
- KS81: value 12 -> =
- KS83: value ENTER -> ENT
- KS84: value RCTRL -> RCTL
- KS85: value RARR -> RAR
- moved KS17 299.3 mm to (151.1, 6.35)
- moved KS81 268.0 mm to (367.0, -16.5)
- moved KS54 203.5 mm to (280.7, -16.5)
- moved KS3 193.8 mm to (108.0, 6.35)
- moved KS60 125.8 mm to (302.3, -16.5)
- moved KS67 119.6 mm to (323.9, -16.5)
- moved KS10 102.5 mm to (129.5, 6.35)
- moved KS74 98.8 mm to (345.4, -16.5)
- moved J1 84.9 mm to (35.7, 84.3)
- moved U1 82.8 mm to (33.8, 103.6), turned to -90 degrees
- moved KS42 2.34 mm to (237.5, -16.5)
- moved KS48 2.25 mm to (259.1, -16.5)
- moved KS30 1.53 mm to (194.3, -16.5)
- moved KS36 0.92 mm to (215.9, -16.5)
- moved KS16 0.46 mm to (151.1, -16.5)
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- renumbered D23 to D22, D28 to D23, D22 to D25, D25 to D26, D26 to D27, D27 to D28, D47 to D48, D48 to D49, D49 to D50, D50 to D51, D51 to D52, D52 to D53, D53 to D54, D54 to D55, D55 to D56, D56 to D57, D57 to D58, D58 to D59, D59 to D60, D60 to D61, D61 to D62, D62 to D63, D63 to D64, D64 to D65, D65 to D66, D66 to D67, D67 to D68, D68 to D69, D69 to D70, D70 to D71, D71 to D72, D72 to D73, D73 to D74, D74 to D75, D75 to D76, D76 to D77, D77 to D78, D78 to D79, D79 to D80, D80 to D81, D81 to D82, D82 to D83, D83 to D84, D84 to D85, D85 to D86, KS23 to KS22, KS28 to KS23, KS22 to KS25, KS25 to KS26, KS86 to KS87
Connections:
- D1 pad 2: ROW0 -> COL0
- D10 pad 2: unconnected-(D10-Pad2) -> COL1
- D11 pad 2: unconnected-(D11-Pad2) -> COL1
- D12 pad 2: unconnected-(D12-Pad2) -> COL1
- D13 pad 2: unconnected-(D13-Pad2) -> COL1
- D14 pad 2: unconnected-(D14-Pad2) -> COL1
- D15 pad 2: ROW0 -> COL2
- D16 pad 2: ROW1 -> COL2
- D17 pad 2: ROW2 -> COL2
- D18 pad 2: ROW3 -> COL2
- D19 pad 2: ROW4 -> COL2
- D2 pad 2: ROW1 -> COL0
- D20 pad 2: ROW5 -> COL2
- D21 pad 2: ROW6 -> COL2
- D22 pad 2: ROW0 -> COL3
- D23 pad 2: ROW1 -> COL3
- D24 pad 2: ROW2 -> COL3
- D25 pad 2: ROW3 -> COL3
- D26 pad 2: ROW4 -> COL3
- D27 pad 2: unconnected-(D26-Pad2) -> COL3
- D28 pad 2: unconnected-(D27-Pad2) -> COL3
- D29 pad 2: ROW0 -> COL4
- D3 pad 2: ROW2 -> COL0
- D30 pad 2: ROW1 -> COL4
- D31 pad 2: ROW2 -> COL4
- D32 pad 2: ROW3 -> COL4
- D33 pad 2: ROW4 -> COL4
- D34 pad 2: ROW6 -> COL4
- D35 pad 2: ROW0 -> COL5
- D36 pad 2: ROW1 -> COL5
- D37 pad 2: ROW2 -> COL5
- D38 pad 2: ROW3 -> COL5
- D39 pad 2: ROW4 -> COL5
- D4 pad 2: ROW3 -> COL0
- D40 pad 2: ROW6 -> COL5
- D41 pad 2: ROW0 -> COL6
- D42 pad 2: ROW1 -> COL6
- D43 pad 2: ROW2 -> COL6
- D44 pad 2: ROW3 -> COL6
- D45 pad 2: ROW4 -> COL6
- D46 pad 2: ROW6 -> COL6
- D48 pad 2: ROW0 -> COL7
- D49 pad 2: ROW1 -> COL7
- D5 pad 2: ROW4 -> COL0
- D50 pad 2: ROW2 -> COL7
- D51 pad 2: ROW3 -> COL7
- D52 pad 2: ROW4 -> COL7
- D53 pad 2: ROW6 -> COL7
- D54 pad 2: ROW0 -> COL8
- D55 pad 2: ROW1 -> COL8
- D56 pad 2: ROW2 -> COL8
- D57 pad 2: ROW3 -> COL8
- D58 pad 2: ROW4 -> COL8
- D59 pad 2: ROW6 -> COL8
- D6 pad 2: ROW5 -> COL0
- D60 pad 2: ROW0 -> COL9
- D61 pad 2: ROW1 -> COL9
- D62 pad 2: ROW2 -> COL9
- D63 pad 2: ROW3 -> COL9
- D64 pad 2: ROW4 -> COL9
- D65 pad 2: ROW5 -> COL9
- D66 pad 2: ROW6 -> COL9
- D67 pad 2: ROW0 -> COL10
- D68 pad 2: ROW1 -> COL10
- D69 pad 2: ROW2 -> COL10
- D7 pad 2: ROW6 -> COL0
- D70 pad 2: ROW3 -> COL10
- D71 pad 2: ROW4 -> COL10
- D72 pad 2: ROW5 -> COL10
- D73 pad 2: ROW6 -> COL10
- D74 pad 2: ROW0 -> COL11
- D75 pad 2: ROW1 -> COL11
- D76 pad 2: ROW2 -> COL11
- D77 pad 2: ROW3 -> COL11
- D78 pad 2: ROW4 -> COL11
- D79 pad 2: ROW5 -> COL11
- D8 pad 2: unconnected-(D8-Pad2) -> COL1
- D80 pad 2: ROW6 -> COL11
- D81 pad 2: ROW0 -> COL12
- D82 pad 2: ROW1 -> COL12
- D83 pad 2: ROW2 -> COL12
- D84 pad 2: ROW3 -> COL12
- D85 pad 2: ROW5 -> COL12
- D86 pad 1: Net-(D85-Pad1) (its old number) -> Net-(D86-Pad1)
- D86 pad 2: ROW6 -> COL12
- D9 pad 2: unconnected-(D9-Pad2) -> COL1
- KS1 pad 1: COL0 -> ROW0
- KS10 pad 1: COL1 -> ROW2
- KS11 pad 1: COL1 -> ROW3
- KS12 pad 1: COL1 -> ROW4
- KS13 pad 1: COL1 -> ROW5
- KS14 pad 1: COL1 -> ROW6
- KS15 pad 1: COL2 -> ROW0
- KS16 pad 1: COL2 -> ROW1
- KS17 pad 1: COL2 -> ROW2
- KS18 pad 1: COL2 -> ROW3
- KS19 pad 1: COL2 -> ROW4
- KS2 pad 1: COL0 -> ROW1
- KS20 pad 1: COL2 -> ROW5
- KS21 pad 1: COL2 -> ROW6
- KS22 pad 1: COL3 -> ROW0
- KS23 pad 1: COL3 -> ROW1
- KS24 pad 1: COL3 -> ROW2
- KS25 pad 1: COL3 -> ROW3
- KS26 pad 1: COL3 -> ROW4
- KS27 pad 1: COL3 -> ROW5
- KS28 pad 1: COL3 -> ROW6
- KS29 pad 1: COL4 -> ROW0
- KS3 pad 1: COL0 -> ROW2
- KS30 pad 1: COL4 -> ROW1
- KS31 pad 1: COL4 -> ROW2
- KS32 pad 1: COL4 -> ROW3
- KS33 pad 1: COL4 -> ROW4
- KS34 pad 1: COL4 -> ROW6
- KS35 pad 1: COL5 -> ROW0
- KS36 pad 1: COL5 -> ROW1
- KS37 pad 1: COL5 -> ROW2
- KS38 pad 1: COL5 -> ROW3
- KS39 pad 1: COL5 -> ROW4
- KS4 pad 1: COL0 -> ROW3
- KS40 pad 1: COL5 -> ROW6
- KS41 pad 1: COL6 -> ROW0
- KS42 pad 1: COL6 -> ROW1
- KS43 pad 1: COL6 -> ROW2
- KS44 pad 1: COL6 -> ROW3
- KS45 pad 1: COL6 -> ROW4
- KS46 pad 1: COL6 -> ROW6
- KS47 pad 1: COL7 -> ROW0
- KS48 pad 1: COL7 -> ROW1
- KS49 pad 1: COL7 -> ROW2
- KS5 pad 1: COL0 -> ROW4
- KS50 pad 1: COL7 -> ROW3
- KS51 pad 1: COL7 -> unconnected-(KS51-Pad1)
- KS52 pad 1: COL7 -> ROW6
- KS53 pad 1: COL8 -> ROW0
- KS54 pad 1: COL8 -> ROW1
- KS55 pad 1: COL8 -> ROW2
- KS56 pad 1: COL8 -> ROW3
- KS57 pad 1: COL8 -> ROW4
- KS58 pad 1: COL8 -> ROW6
- KS59 pad 1: COL9 -> ROW0
- KS6 pad 1: COL0 -> ROW5
- KS60 pad 1: COL9 -> ROW1
- KS61 pad 1: COL9 -> ROW2
- KS62 pad 1: COL9 -> ROW3
- KS63 pad 1: COL9 -> ROW4
- KS64 pad 1: COL9 -> ROW5
- KS65 pad 1: COL9 -> ROW6
- KS66 pad 1: COL10 -> ROW0
- KS67 pad 1: COL10 -> ROW1
- KS68 pad 1: COL10 -> ROW2
- KS69 pad 1: COL10 -> ROW3
- KS7 pad 1: COL0 -> ROW6
- KS70 pad 1: COL10 -> ROW4
- KS71 pad 1: COL10 -> ROW5
- KS72 pad 1: COL10 -> ROW6
- KS73 pad 1: COL11 -> ROW0
- KS74 pad 1: COL11 -> ROW1
- KS75 pad 1: COL11 -> ROW2
- KS76 pad 1: COL11 -> ROW3
- KS77 pad 1: COL11 -> ROW4
- KS78 pad 1: COL11 -> ROW5
- KS79 pad 1: COL11 -> ROW6
- KS8 pad 1: COL1 -> ROW0
- KS80 pad 1: COL12 -> ROW0
- KS81 pad 1: COL12 -> ROW1
- KS82 pad 1: COL12 -> ROW2
- KS83 pad 1: COL12 -> ROW3
- KS84 pad 1: COL12 -> ROW5
- KS85 pad 1: COL12 -> ROW6
- KS85 pad 2: Net-(D85-Pad1) (its old number) -> Net-(D86-Pad1)
- KS87 pad 1: COL13 -> ROW2
- KS87 pad 2: COL12 -> Net-(D88-Pad1)
- KS9 pad 1: COL1 -> ROW1
- SW1 pad 2: Net-(D86-Pad1) -> Net-(D87-Pad1)
- SW1 pad C: GND -> unconnected-(SW1-PadC)
- U1 pad 1: ROW0 -> unconnected-(U1-Pad1)
- U1 pad 10: COL2 -> unconnected-(U1-Pad10)
- U1 pad 11: COL3 -> unconnected-(U1-Pad11)
- U1 pad 12: COL4 -> unconnected-(U1-Pad12)
- U1 pad 15: unconnected-(U1-Pad15) -> GND
- U1 pad 18: COL5 -> unconnected-(U1-Pad18)
- U1 pad 19: SDA -> unconnected-(U1-Pad19)
- U1 pad 20: SCL -> unconnected-(U1-Pad20)
- U1 pad 21: COL6 -> unconnected-(U1-Pad21)
- U1 pad 22: COL7 -> unconnected-(U1-Pad22)
- U1 pad 23: unconnected-(U1-Pad23) -> GND
- U1 pad 26: COL9 -> unconnected-(U1-Pad26)
- U1 pad 27: COL10 -> unconnected-(U1-Pad27)
- U1 pad 28: COL11 -> unconnected-(U1-Pad28)
- U1 pad 29: COL12 -> unconnected-(U1-Pad29)
- U1 pad 3: Net-(J1-Pad2) -> /D-
- U1 pad 30: COL13 -> unconnected-(U1-Pad30)
- U1 pad 31: ROW1 -> unconnected-(U1-Pad31)
- U1 pad 32: ROW2 -> unconnected-(U1-Pad32)
- U1 pad 35: unconnected-(U1-Pad35) -> GND
- U1 pad 36: ROW3 -> unconnected-(U1-Pad36)
- U1 pad 37: ROW4 -> unconnected-(U1-Pad37)
- U1 pad 38: ROW5 -> unconnected-(U1-Pad38)
- U1 pad 39: ROW6 -> unconnected-(U1-Pad39)
- U1 pad 4: Net-(J1-Pad3) -> /D+
- U1 pad 43: unconnected-(U1-Pad43) -> GND
- U1 pad 5: unconnected-(U1-Pad5) -> GND
- U1 pad 8: COL0 -> unconnected-(U1-Pad8)
- U1 pad 9: COL1 -> unconnected-(U1-Pad9)

Commit message: stuff
Parts:
- U1: moved to B.Cu
- moved U1 168.2 mm to (50.2, -63.8)
- moved J1 164.1 mm to (48.2, -79.3), turned to 180 degrees
- moved D87 67.3 mm to (89.1, -87.2)
- moved D47 66.6 mm to (76.5, -92.3)
- moved KS80 48.5 mm to (357.1, -63.4)
- moved KS73 45.5 mm to (338.1, -63.4)
- moved KS66 43.5 mm to (319.1, -63.4)
- moved KS59 41.0 mm to (300.0, -63.4)
- moved SW1 40.8 mm to (396.4, -63.6)
- moved SW1 37.6 mm to (84.6, 30.1)
- moved KS53 33.9 mm to (270.9, -63.4)
- moved KS23 33.4 mm to (145.7, -36.4)
- moved KS16 31.9 mm to (126.1, -36.4)
- moved KS47 30.6 mm to (251.8, -63.4)
- moved KS9 29.9 mm to (107.2, -36.4)
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Connections:
- J1 pad A6: unconnected-(J1-PadA6) -> D+
- J1 pad A7: unconnected-(J1-PadA7) -> D-
- J1 pad B6: /D+ -> unconnected-(J1-PadB6)
- J1 pad B7: /D- -> unconnected-(J1-PadB7)
- U1 pad 1: unconnected-(U1-Pad1) -> ROW0
- U1 pad 10: unconnected-(U1-Pad10) -> COL2
- U1 pad 11: unconnected-(U1-Pad11) -> COL3
- U1 pad 12: unconnected-(U1-Pad12) -> COL4
- U1 pad 18: unconnected-(U1-Pad18) -> COL5
- U1 pad 19: unconnected-(U1-Pad19) -> SDA
- U1 pad 20: unconnected-(U1-Pad20) -> SCL
- U1 pad 21: unconnected-(U1-Pad21) -> COL6
- U1 pad 22: unconnected-(U1-Pad22) -> COL7
- U1 pad 26: unconnected-(U1-Pad26) -> COL9
- U1 pad 27: unconnected-(U1-Pad27) -> COL10
- U1 pad 28: unconnected-(U1-Pad28) -> COL11
- U1 pad 29: unconnected-(U1-Pad29) -> COL12
- U1 pad 3: /D- -> D-
- U1 pad 30: unconnected-(U1-Pad30) -> COL13
- U1 pad 31: unconnected-(U1-Pad31) -> ROW1
- U1 pad 32: unconnected-(U1-Pad32) -> ROW2
- U1 pad 36: unconnected-(U1-Pad36) -> ROW3
- U1 pad 37: unconnected-(U1-Pad37) -> ROW4
- U1 pad 38: unconnected-(U1-Pad38) -> ROW5
- U1 pad 39: unconnected-(U1-Pad39) -> ROW6
- U1 pad 4: /D+ -> D+
- U1 pad 8: unconnected-(U1-Pad8) -> COL0
- U1 pad 9: unconnected-(U1-Pad9) -> COL1
Routing:
- net D-: track 0.00 -> 9.99 mm
- net D+: track 0.00 -> 9.99 mm
