File: Keyboard/Keyboard.kicad_sch (KiCad schematic)
At the start: 177 parts, among them J1 Conn_01x06, J2 Conn_01x04, J3 Conn_01x16

Commit message: Finished First Pass of Schematic and Layout
Parts:
- removed J1: Conn_01x06, Connector_PinHeader_2.54mm:PinHeader_1x06_P2.54mm_Vertical, symbol Connector_Generic:Conn_01x06
- removed J3: Conn_01x16, Connector_PinHeader_2.54mm:PinHeader_1x16_P2.54mm_Vertical, symbol Connector_Generic:Conn_01x16
- added J4: Conn_02x20_Odd_Even, Keyboard:SAMTEC_ERF8-020-05.0-L-DV-K-TR, symbol Connector_Generic:Conn_02x20_Odd_Even
- added R1, R10, R11, R12, R13, R2, R3, R4, R5, R6, R7, R8, R9: 10k, Resistor_SMD:R_0805_2012Metric_Pad1.20x1.40mm_HandSolder, symbol Device:R_Small_US
- added S1: PEC12R-4220F-S0024, Keyboard:XDCR_PEC12R-4220F-S0024, symbol Keyboard:PEC12R-4220F-S0024
- D1, D10, D11, D12, D13, D14, D15, D16, D17, D18, D19, D2, D20, D21, D22, D23, D24, D25, D26, D27, D28, D29, D3, D30, D31, D32, D33, D34, D35, D36, D37, D38, D39, D4, D40, D41, D42, D43, D44, D45, D46, D47, D48, D49, D5, D50, D51, D52, D53, D54, D55, D56, D57, D58, D59, D6, D60, D61, D62, D63, D64, D65, D66, D67, D68, D69, D7, D70, D71, D72, D73, D74, D75, D76, D77, D78, D79, D8, D80, D81, D82, D83, D84, D9: footprint Diode_SMD:D_0805_2012Metric -> Diode_SMD:D_0805_2012Metric_Pad1.15x1.40mm_HandSolder
Connections:
- net COL0: now also J4.31 (Pin_31)
- net COL1: now also J4.29 (Pin_29)
- net COL10: now also J4.11 (Pin_11)
- net COL11: now also J4.09 (Pin_9)
- net COL12: now also J4.07 (Pin_7)
- net COL13: now also J4.05 (Pin_5)
- net COL14: now also J4.03 (Pin_3)
- net COL15: now also J4.01 (Pin_1)
- net COL2: now also J4.27 (Pin_27)
- net COL3: now also J4.25 (Pin_25)
- net COL4: now also J4.23 (Pin_23)
- net COL5: now also J4.21 (Pin_21)
- net COL6: now also J4.19 (Pin_19)
- net COL7: now also J4.17 (Pin_17)
- net COL8: now also J4.15 (Pin_15)
- net COL9: now also J4.13 (Pin_13)
- net GND: now also J4.33 (Pin_33), J4.35 (Pin_35), J4.37 (Pin_37), J4.39 (Pin_39), R1.2, R10.2, R12.2, R4.2, R6.2, R8.2, S1.2, S1.C (COMMON), S1.SH1 (SHIELD), S1.SH2 (SHIELD__1)
- net ROW0: now also J4.12 (Pin_12), R1.1, R2.2
- net ROW1: now also J4.10 (Pin_10), R3.2, R4.1
- net ROW2: now also J4.08 (Pin_8), R5.2, R6.1
- net ROW3: now also J4.06 (Pin_6), R7.2, R8.1
- net ROW4: now also J4.04 (Pin_4), R10.1, R9.2
- net ROW5: now also J4.02 (Pin_2), R11.2, R12.1
- net VCC: now also J4.34 (Pin_34), J4.36 (Pin_36), J4.38 (Pin_38), J4.40 (Pin_40), R11.1, R13.1, R2.1, R3.1, R5.1, R7.1, R9.1
- new net ENC_A: J4.16 (Pin_16), S1.A (CHANNEL_A)
- new net ENC_B: J4.14 (Pin_14), S1.B (CHANNEL_B)
- new net ENC_SW: J4.18 (Pin_18), R13.2, S1.1
