File: CustomKeyboard.kicad_pcb (KiCad board)
At the start: 2 copper layers, 308 x 117.5 mm, 168 parts, among them SW1 ESC, SW10 F9, SW11 F10, SW12 F11, SW13 F12, SW14 PrtSc/NmLk, SW15 Pause/ScrLk, SW16 Delete/Insert, SW18 1, SW19 2, SW2 F1, SW20 3, SW21 4, SW22 5, SW23 6, SW24 7, SW25 8, SW26 9, SW27 0, SW28 -, SW29 =, SW3 F2, SW30 Backspace, SW31 Home, SW32 Tab, SW33 Q, SW34 W, SW35 E, SW36 R, SW37 T, SW38 Y, SW39 U, SW4 F3, SW40 I, SW41 O, SW42 P, SW43 [, SW44 ], SW45 \, SW46 PgUp, SW47 CapsLock, SW48 A, SW49 S, SW5 F4, SW50 D, SW51 F, SW52 G, SW53 H, SW54 J, SW55 K, SW56 L, SW57 ;, SW58 ', SW59 Enter, SW6 F5, SW60 PgDn, SW61 LShift, SW62 Z, SW63 X, SW64 C, SW65 V, SW66 B, SW67 N, SW68 M, SW69 ,, SW7 F6, SW70 ., SW71 /, SW72 RShift, SW73 Up, SW74 End, SW75 CTRL, SW76 Win, SW77 Alt, SW78 Space, SW79 Alt, SW8 F7, SW80 Fn, SW81 Ctrl, SW82 Left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

Commit message: Complete rework with hot swap sockets and high density pin board to board connectors
Parts:
- added H1: MountingHole, MountingHole:MountingHole_3.2mm_M3_Pad_Via, F.Cu at (362.0, 75.0)
- added H2: MountingHole, MountingHole:MountingHole_3.2mm_M3_Pad_Via, F.Cu at (362.0, 193.0)
- added H3: MountingHole, MountingHole:MountingHole_3.2mm_M3_Pad_Via, F.Cu at (45.0, 193.0)
- added H4: MountingHole, MountingHole:MountingHole_3.2mm_M3_Pad_Via, F.Cu at (45.0, 75.0)
- added J1: Conn_02x16_Odd_Even, keyboard-fps:HRS_DF12NB_3.0_-32DS-0.5V_51_, B.Cu at (59.7, 77.0)
- added J2: Conn_02x16_Odd_Even, keyboard-fps:HRS_DF12NB_3.0_-32DS-0.5V_51_, B.Cu at (345.5, 77.0)
- added R1: 10k, Resistor_SMD:R_0805_2012Metric_Pad1.20x1.40mm_HandSolder, B.Cu at (67.5, 82.5)
- added R10: 10k, Resistor_SMD:R_0805_2012Metric_Pad1.20x1.40mm_HandSolder, B.Cu at (237.5, 81.0)
- added R11: 10k, Resistor_SMD:R_0805_2012Metric_Pad1.20x1.40mm_HandSolder, B.Cu at (256.5, 81.0)
- added R12: 10k, Resistor_SMD:R_0805_2012Metric_Pad1.20x1.40mm_HandSolder, B.Cu at (275.5, 81.0)
- added R13: 10k, Resistor_SMD:R_0805_2012Metric_Pad1.20x1.40mm_HandSolder, B.Cu at (295.0, 81.0)
- added R14: 10k, Resistor_SMD:R_0805_2012Metric_Pad1.20x1.40mm_HandSolder, B.Cu at (314.0, 81.0)
- added R15: 10k, Resistor_SMD:R_0805_2012Metric_Pad1.20x1.40mm_HandSolder, B.Cu at (332.5, 81.0)
- added R16: 10k, Resistor_SMD:R_0805_2012Metric_Pad1.20x1.40mm_HandSolder, B.Cu at (351.5, 81.0)
- added R2: 10k, Resistor_SMD:R_0805_2012Metric_Pad1.20x1.40mm_HandSolder, B.Cu at (86.0, 82.0)
- added R3: 10k, Resistor_SMD:R_0805_2012Metric_Pad1.20x1.40mm_HandSolder, B.Cu at (104.5, 81.5)
- added R4: 10k, Resistor_SMD:R_0805_2012Metric_Pad1.20x1.40mm_HandSolder, B.Cu at (124.0, 81.0)
- added R5: 10k, Resistor_SMD:R_0805_2012Metric_Pad1.20x1.40mm_HandSolder, B.Cu at (142.5, 81.0)
- added R6: 10k, Resistor_SMD:R_0805_2012Metric_Pad1.20x1.40mm_HandSolder, B.Cu at (161.5, 81.0)
- added R7: 10k, Resistor_SMD:R_0805_2012Metric_Pad1.20x1.40mm_HandSolder, B.Cu at (180.5, 81.0)
- added R8: 10k, Resistor_SMD:R_0805_2012Metric_Pad1.20x1.40mm_HandSolder, B.Cu at (199.5, 81.0)
- added R9: 10k, Resistor_SMD:R_0805_2012Metric_Pad1.20x1.40mm_HandSolder, B.Cu at (219.0, 81.0)
- D25, D26, D27, D28, D29, D30, D31, D32, D33, D34, D35, D36, D37, D38, D39, D40, D41, D42, D43, D44, D45, D46, D47, D48, D49, D50, D51, D52, D53, D54, D55, D56, D57, D58, D59, D60, D61, D62, D63, D64, D65, D66, D67, D68, D69, D70, D71, D72, D73, D74, D75, D76, D77, D78, D79, D80, D81, D82, D83, D84: moved to B.Cu
- moved D47 9.27 mm to (76.0, 150.5), turned to 90 degrees
- moved D74 9.25 mm to (354.5, 170.0), turned to 90 degrees
- moved D71 9.20 mm to (283.0, 170.0), turned to 90 degrees
- moved D75 9.12 mm to (71.0, 189.0), turned to 90 degrees
- moved D61 9.10 mm to (80.5, 170.0), turned to 90 degrees
- moved D63 9.10 mm to (130.5, 170.0), turned to 90 degrees
- moved D48 9.09 mm to (102.0, 150.5), turned to 90 degrees
- moved D78 9.06 mm to (190.0, 189.0), turned to 90 degrees
- moved D39 9.05 mm to (211.5, 131.5), turned to 90 degrees
- moved D64 9.04 mm to (149.5, 170.0), turned to 90 degrees
- moved D25 9.04 mm to (221.0, 112.5), turned to 90 degrees
- moved D49 9.03 mm to (121.0, 150.5), turned to 90 degrees
- moved D40 9.00 mm to (230.5, 131.5), turned to 90 degrees
- moved D72 9.00 mm to (309.0, 170.0), turned to 90 degrees
- moved D65 9.00 mm to (168.5, 170.0), turned to 90 degrees
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Connections:
- net Net-(SW1-Pad1) renamed /COL1
- net Net-(SW10-Pad1) renamed /COL10
- net Net-(SW11-Pad1) renamed /COL11
- net Net-(SW12-Pad1) renamed /COL12
- net Net-(SW13-Pad1) renamed /COL13
- net Net-(SW14-Pad1) renamed /COL14
- net Net-(SW15-Pad1) renamed /COL15
- net Net-(SW16-Pad1) renamed /COL16
- net Net-(SW18-Pad1) renamed /COL2
- net Net-(SW19-Pad1) renamed /COL3
- net Net-(SW20-Pad1) renamed /COL4
- net Net-(SW21-Pad1) renamed /COL5
- net Net-(SW22-Pad1) renamed /COL6
- net Net-(SW23-Pad1) renamed /COL7
- net Net-(SW24-Pad1) renamed /COL8
- net Net-(SW25-Pad1) renamed /COL9
Routing:
- net /ROW6: track 0.00 -> 426.3 mm
- net /ROW5: track 0.00 -> 406.8 mm
- net /COL16: track 0.00 -> 395.4 mm, vias 0 -> 7
- net /COL15: track 0.00 -> 394.4 mm, vias 0 -> 7
- net /ROW4: track 0.00 -> 386.3 mm
- net /ROW3: track 0.00 -> 364.7 mm
- net /COL14: track 0.00 -> 355.6 mm, vias 0 -> 3
- net /ROW2: track 0.00 -> 343.8 mm
- net /COL12: track 0.00 -> 336.0 mm, vias 0 -> 7
- net /ROW1: track 0.00 -> 324.8 mm
- net +3.3V: track 0.00 -> 319.8 mm, vias 0 -> 2
- net GND: track 0.00 -> 316.7 mm, vias 0 -> 2
- net /COL11: track 0.00 -> 309.7 mm, vias 0 -> 7
- net /COL10: track 0.00 -> 289.2 mm, vias 0 -> 7
- net /COL13: track 0.00 -> 283.0 mm, vias 0 -> 4
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Other:
- board size 308 x 117.5 mm -> 327 x 128 mm
